Commit message: add the library description and import the hardware interface

File: ros2_pkg/src/ruche_ros2_control/description/ros2_control/diffelegoo.ros2_control.xacro (robot description, xacro)
@@ -29,5 +29,22 @@
         <!-- Case: real hardware -->
         <xacro:unless value="$(arg simulate)">
-            <!-- TODO: Insert hardware interface here -->
+            <hardware>
+                <plugin>ruche_ros2_control/ElegooBt2SerialHardware</plugin>
+                <param name="left_wheel_name">wheel_l_joint</param>
+                <param name="right_wheel_name">wheel_r_joint</param>
+                <param name="device_id">58:BF:25:9D:CD:F6</param>
+            </hardware>
+            <joint name="wheel_l_joint">
+                <command_interface name="velocity">
+                    <param name="min">-10</param>
+                    <param name="max">10</param>
+                </command_interface>
+            </joint>
+            <joint name="wheel_r_joint">
+                <command_interface name="velocity">
+                    <param name="min">-10</param>
+                    <param name="max">10</param>
+                </command_interface>
+            </joint>
         </xacro:unless>
     </xacro:macro>

Commit message: Fixes #16. Enhable the import of a basic  (empty) hardware interface

File: ros2_pkg/src/ruche_ros2_control/description/ros2_control/diffelegoo.ros2_control.xacro (robot description, xacro)
@@ -29,22 +29,23 @@
         <!-- Case: real hardware -->
         <xacro:unless value="$(arg simulate)">
+            <ros2_control  name="ElegooSystem" type="system">
             <hardware>
                 <plugin>ruche_ros2_control/ElegooBt2SerialHardware</plugin>
-                <param name="left_wheel_name">wheel_l_joint</param>
-                <param name="right_wheel_name">wheel_r_joint</param>
-                <param name="device_id">58:BF:25:9D:CD:F6</param>
+                <param name="p1">0</param>
+                <param name="p2">3.0</param>
             </hardware>
             <joint name="wheel_l_joint">
-                <command_interface name="velocity">
-                    <param name="min">-10</param>
-                    <param name="max">10</param>
-                </command_interface>
+                <command_interface name="velocity"/>
+                <!-- No state interface are provided, but declared to start the joint_state_broadcaster -->
+                <state_interface name="position"/>
+                <state_interface name="velocity"/>
             </joint>
             <joint name="wheel_r_joint">
-                <command_interface name="velocity">
-                    <param name="min">-10</param>
-                    <param name="max">10</param>
-                </command_interface>
+                <command_interface name="velocity"/>
+                <!-- No state interface are provided, but declared to start the joint_state_broadcaster -->
+                <state_interface name="position"/>
+                <state_interface name="velocity"/>
             </joint>
+            </ros2_control>
         </xacro:unless>
     </xacro:macro>

File: ros2_pkg/src/ruche_ros2_control/description/urdf/diffelegoo.urdf.xacro (robot description, xacro)
@@ -1,9 +1,9 @@
 <?xml version="1.0"?>
-<robot xmlns:xacro="http://www.ros.org/wiki/xacro"  name="$(arg robot_name)">
+<robot xmlns:xacro="http://www.ros.org/wiki/xacro" name="$(arg robot_name)">
     <!-- Define input arguments -->
-    <xacro:arg name="simulate" default="true"/>
+    <xacro:arg name="simulate" default="true" />
     <!-- Define parameters -->
     <xacro:property name="name" value="$(arg robot_name)" />
-     <!-- Include other xacro files here -->
+    <!-- Include other xacro files here -->
     <xacro:include filename="inertial_calculations.xacro" />
     <xacro:include filename="${name}_materials.xacro" />
@@ -11,8 +11,8 @@
     <!-- Load ros2 and gazebo plugins -->
     <xacro:include filename="${name}.ros2_control.xacro" />
-    <xacro:robot_ros2_control/>
+    <xacro:robot_ros2_control />
     <xacro:if value="$(arg simulate)">
         <xacro:include filename="${name}_gazebo.xacro" />
-        <xacro:diffbot_gazebo/>
+        <xacro:diffbot_gazebo />
     </xacro:if>
     <!-- Base link -->
@@ -20,96 +20,101 @@
     <!-- Position of the chassis link with respect to the base link -->
     <joint name="chassis_joint" type="fixed">
-        <origin xyz="0.01 0 0" rpy="0 0 0"/>
-        <parent link="base_link"/>
-        <child link="chassis_link"/>
+        <origin xyz="0.01 0 0" rpy="0 0 0" />
+        <parent link="base_link" />
+        <child link="chassis_link" />
     </joint>
     <!-- Chassis -->
     <link name="chassis_link">
         <visual>
-            <origin xyz="${base_width/2 - wheel_x_from_back} 0 ${base_height/2-wheel_z_from_base}" rpy="0 0 0"/>
+            <origin xyz="${base_width/2 - wheel_x_from_back} 0 ${base_height/2-wheel_z_from_base}"
+                rpy="0 0 0" />
             <geometry>
-                <box size="${base_width} ${base_depth} ${base_height}"/>
+                <box size="${base_width} ${base_depth} ${base_height}" />
             </geometry>
             <material name="red" />
         </visual>
         <collision>
-            <origin xyz="${base_width/2 - wheel_x_from_back} 0 ${base_height/2-wheel_z_from_base}" rpy="0 0 0"/>
+            <origin xyz="${base_width/2 - wheel_x_from_back} 0 ${base_height/2-wheel_z_from_base}"
+                rpy="0 0 0" />
             <geometry>
-                <box size="${base_width} ${base_depth} ${base_height}"/>
+                <box size="${base_width} ${base_depth} ${base_height}" />
             </geometry>
         </collision>
-        <xacro:inertial_box mass="${base_mass}" x="${base_width}" y="${base_depth}" z="${base_height}">
-            <origin xyz="${base_width/2 - wheel_x_from_back} 0 ${base_height/2-wheel_z_from_base}" rpy="0 0 0"/>
+        <xacro:inertial_box mass="${base_mass}" x="${base_width}" y="${base_depth}"
+            z="${base_height}">
+            <origin xyz="${base_width/2 - wheel_x_from_back} 0 ${base_height/2-wheel_z_from_base}"
+                rpy="0 0 0" />
         </xacro:inertial_box>
     </link>
     <joint name="wheel_l_joint" type="continuous">
-        <origin xyz="0 ${base_depth/2+wheel_height+0.005} 0" rpy="${pi/2} 0 0"/>
-        <parent link="base_link"/>
-        <child link="wheel_l_link"/>
-        <axis xyz="0 0 -1"/>
+        <origin xyz="0 ${base_depth/2+wheel_height+0.005} 0" rpy="${pi/2} 0 0" />
+        <parent link="base_link" />
+        <child link="wheel_l_link" />
+        <axis xyz="0 0 -1" />
     </joint>
     <link name="wheel_l_link">
         <visual>
-            <origin xyz="0 0 ${wheel_height/2}" rpy="0 0 0"/>
+            <origin xyz="0 0 ${wheel_height/2}" rpy="0 0 0" />
             <geometry>
-                <cylinder radius="${wheel_r}" length="${wheel_height}"/>
+                <cylinder radius="${wheel_r}" length="${wheel_height}" />
             </geometry>
             <material name="black" />
         </visual>
         <collision>
-            <origin xyz="0 0 ${wheel_height/2}" rpy="0 0 0"/>
+            <origin xyz="0 0 ${wheel_height/2}" rpy="0 0 0" />
             <geometry>
-                <cylinder radius="${wheel_r}" length="${wheel_height}"/>
+                <cylinder radius="${wheel_r}" length="${wheel_height}" />
             </geometry>
         </collision>
         <xacro:inertial_cylinder mass="${wheel_mass}" r="${wheel_r}" h="${wheel_height}">
-            <origin xyz="0 0 0" rpy="0 0 0"/>
+            <origin xyz="0 0 0" rpy="0 0 0" />
         </xacro:inertial_cylinder>
     </link>
     <joint name="wheel_r_joint" type="continuous">
-        <origin xyz="0 -${base_depth/2+0.005} 0" rpy="${pi/2} 0 0"/>
-        <parent link="base_link"/>
-        <child link="wheel_r_link"/>
-        <axis xyz="0 0 -1"/>
+        <origin xyz="0 -${base_depth/2+0.005} 0" rpy="${pi/2} 0 0" />
+        <parent link="base_link" />
+        <child link="wheel_r_link" />
+        <axis xyz="0 0 -1" />
     </joint>
     <link name="wheel_r_link">
         <visual>
-            <origin xyz="0 0 ${wheel_height/2}" rpy="0 0 0"/>
+            <origin xyz="0 0 ${wheel_height/2}" rpy="0 0 0" />
             <geometry>
-                <cylinder radius="${wheel_r}" length="${wheel_height}"/>
+                <cylinder radius="${wheel_r}" length="${wheel_height}" />
             </geometry>
             <material name="black" />
         </visual>
         <collision>
-            <origin xyz="0 0 ${wheel_height/2}" rpy="0 0 0"/>
+            <origin xyz="0 0 ${wheel_height/2}" rpy="0 0 0" />
             <geometry>
-                <cylinder radius="${wheel_r}" length="${wheel_height}"/>
+                <cylinder radius="${wheel_r}" length="${wheel_height}" />
             </geometry>
         </collision>
         <xacro:inertial_cylinder mass="${wheel_mass}" r="${wheel_r}" h="${wheel_height}">
-            <origin xyz="0 0 0" rpy="0 0 0"/>
+            <origin xyz="0 0 0" rpy="0 0 0" />
         </xacro:inertial_cylinder>
     </link>
     <joint name="caster_joint" type="fixed">
-        <origin xyz="${base_width - wheel_x_from_back - caster_r} 0 ${-wheel_r + caster_r}" rpy="0 0 0"/>
-        <parent link="chassis_link"/>
-        <child link="caster_link"/>
+        <origin xyz="${base_width - wheel_x_from_back - caster_r} 0 ${-wheel_r + caster_r}"
+            rpy="0 0 0" />
+        <parent link="chassis_link" />
+        <child link="caster_link" />
     </joint>
     <link name="caster_link">
         <visual>
-            <origin xyz="0 0 0" rpy="0 0 0"/>
+            <origin xyz="0 0 0" rpy="0 0 0" />
             <geometry>
-                <sphere radius="${caster_r}"/>
+                <sphere radius="${caster_r}" />
             </geometry>
             <material name="gray" />
         </visual>
         <collision>
-            <origin xyz="0 0 0" rpy="0 0 0"/>
+            <origin xyz="0 0 0" rpy="0 0 0" />
             <geometry>
-                <sphere radius="${caster_r}"/>
+                <sphere radius="${caster_r}" />
             </geometry>
         </collision>
         <xacro:inertial_sphere mass="${caster_mass}" r="${wheel_r}">
-            <origin xyz="0 0 0" rpy="0 0 0"/>
+            <origin xyz="0 0 0" rpy="0 0 0" />
         </xacro:inertial_sphere>
     </link>
